Commit message: Urdf changed

File: cfg/arm_model/so101_new_calib.urdf (robot description, URDF)
Before this commit: robot so101_new_calib, 9 links, 8 joints
Joints:
- joint key_contact_frame_joint: origin xyz=0.001 -0.001 0.006 rpy=0 0 0 -> xyz=0.00 0.00 0.006 rpy=0 0 0

Commit message: parameters tuning and gemini backend addition to the branch

File: cfg/arm_model/so101_new_calib.urdf (robot description, URDF)
Before this commit: robot so101_new_calib, 9 links, 8 joints
Joints:
- joint key_contact_frame_joint: origin xyz=0.00 0.00 0.006 rpy=0 0 0 -> xyz=0.00 0.00 0.010 rpy=0 0 0

Commit message: parameters tuned and updated

File: cfg/arm_model/so101_new_calib.urdf (robot description, URDF)
Before this commit: robot so101_new_calib, 9 links, 8 joints
Joints:
- joint key_contact_frame_joint: origin xyz=0.00 0.00 0.010 rpy=0 0 0 -> xyz=-0.002 -0.005 0.0055 rpy=0 0 0

Commit message: tunnnnnnnnnnnnong

File: cfg/arm_model/so101_new_calib.urdf (robot description, URDF)
Before this commit: robot so101_new_calib, 9 links, 8 joints
Joints:
- joint key_contact_frame_joint: origin xyz=-0.002 -0.005 0.0055 rpy=0 0 0 -> xyz=-0.002 -0.005 0.01 rpy=0 0 0
